File: kicad/gpsv1.1/gpsv1.1.kicad_pcb (KiCad board)
At the start: 2 copper layers, 100 x 100 mm, 22 parts, among them J1 Conn_01x01_Female, J2 Conn_01x01_Female, J3 Conn_01x01_Female

Commit message: Made sensors work
Parts:
- removed G***: LOGO, Custom_sym:K-State Logo
- removed J1, J2, J3: Conn_01x01_Female, Custom_sym:1x1 Pad
- removed MAG1: Magnetometer, Custom_sym:Magnetometer
- added Ant1: SMAAntennaMale, Custom_sym:SMAAntennaMale, F.Cu at (300.0, 67.5)
- added DC-DC1: BuckConverter(LM2596), Custom_sym:BuckConverter(LM2596), F.Cu at (155.0, 100.0)
- added REF**: 1×20, Custom_sym:1×20, F.Cu at (183.8, 132.0)
- added REF**: 1×20, Custom_sym:1×20, F.Cu at (182.5, 130.0)
- added REF**: 1×24, Custom_sym:1×24, F.Cu at (252.6, 136.5)
- added REF**: 1×24, Custom_sym:1×24, F.Cu at (252.6, 156.8)
- added Rasp1: RaspberryPi3, Custom_sym:RasberryPI3, F.Cu at (177.5, 117.5)
- added U1: ExternalBattery, Custom_sym:ExternalBattery, F.Cu at (117.5, 80.0)
- added XH-3A1: XH-3AFemaleConnector, Custom_sym:XH-3A Female Connector, F.Cu at (285.0, 62.5)
- added XH-3A2: XH-3AFemaleConnector, Custom_sym:XH-3A Female Connector, F.Cu at (267.5, 62.5)
- added XH-3A3: XH-3AFemaleConnector, Custom_sym:XH-3A Female Connector, F.Cu at (142.5, 62.5)
- added XH-3A4: XH-3AFemaleConnector, Custom_sym:XH-3A Female Connector, F.Cu at (160.0, 62.5)
- moved Teensy1 173.5 mm to (242.5, 151.7), turned to 270 degrees
- moved TOF3 172.4 mm to (296.0, 133.0)
- moved R7 168.0 mm to (288.5, 145.5)
- moved R5 167.7 mm to (288.5, 130.5)
- moved PA1 164.0 mm to (275.0, 95.0)
- moved R6 163.6 mm to (278.5, 180.5), turned to 45 degrees
- moved TOF4 159.5 mm to (281.0, 188.0), turned to 45 degrees
- moved R8 152.8 mm to (268.5, 190.5), turned to 45 degrees
- moved R9 135.3 mm to (213.5, 195.5)
- moved TOF5 134.6 mm to (211.0, 203.0)
- moved R10 134.4 mm to (198.5, 195.5)
- moved TOF1 113.4 mm to (141.0, 188.0), turned to 315 degrees
- moved R1 110.3 mm to (156.0, 190.5), turned to 135 degrees
- moved R3 103.7 mm to (146.0, 180.5), turned to 135 degrees
- moved TOF2 99.4 mm to (126.0, 133.0)
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Connections:
- net Gnd renamed GND
- net Vin renamed 5V
Routing:
- net DIR1: track 0.00 -> 145.2 mm
- net PWMRight: track 0.00 -> 114.6 mm
- net PWMLeft: track 0.00 -> 109.8 mm
- net DIR2: track 0.00 -> 98.1 mm
- net GND: track 2.33 -> 99.0 mm, vias 1 -> 5
- net Net-(R5-Pad1): track 34.1 -> 99.7 mm
- net SCL: track 57.0 -> 2.56 mm
- net Trig1: track 56.6 -> 105.4 mm
- net Trig2: track 43.7 -> 92.5 mm
- net SDA: track 50.7 -> 2.56 mm
- net Net-(R6-Pad1): track 40.0 -> 87.5 mm
- net Net-(R1-Pad2): track 31.9 -> 72.6 mm
- net Net-(R2-Pad2): track 39.4 -> 79.3 mm
- net Trig4: track 43.8 -> 83.3 mm
- net Trig5: track 55.3 -> 87.2 mm
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Other:
- board size 100 x 100 mm -> 200 x 150.5 mm
- board text removed: "KSU Robotics AVC Team"
