File: kicad/gpsv1.1/gpsv1.1.sch (KiCad schematic (older format))
At the start: 16 parts

Commit message: 20-21
Parts:
- added U?: UltimateGPS, symbol custom_sym:UltimateGPS
Connections:
- net Gnd: now also R?.1, R?.1, R?.1, R?.2, R?.2; no longer R?.1, R?.1, R?.1, R?.1, R?.1, R?.2, R?.2, R?.2, R?.2, R?.2
- net at T?.30: now also R?.1, R?.2; no longer R?.2
- net at T?.32: now also R?.1, R?.2; no longer R?.2
- net at T?.34: now also R?.1, R?.2; no longer R?.1
- net at T?.36: now also R?.1, R?.2; no longer R?.1
- net at T?.38: now also R?.1, R?.2; no longer R?.1
- net at T?.~ (GND): now also U?.~ (GND)
- new net: T?.~ (GND), U?.~ (GND) (x3)
Other:
- moved on the sheet: R?, U?

Commit message: Made the pcb
Parts:
- removed U?: UltimateGPS, symbol custom_sym:UltimateGPS
- added J1, J2, J3: Conn_01x01_Female, Custom_sym:1x1 Pad, symbol Connector:Conn_01x01_Female
- added MAG1: Magnetometer, Custom_sym:Magnetometer, symbol custom_sym:Magnetometer
- added PA1: PA1616D, Custom_sym:GPS PA1616D, symbol custom_sym:PA1616D
- R1, R10, R2, R3, R4, R5, R6, R7, R8, R9: renamed from R?; footprint (none) -> Resistors_THT:R_Axial_DIN0207_L6.3mm_D2.5mm_P10.16mm_Horizontal
- TOF1, TOF2, TOF3, TOF4, TOF5: renamed from U?; footprint (none) -> Custom_sym:TOF Sensor
- Teensy1: renamed from T?; footprint (none) -> Custom_sym:Teensy 4.1
Connections:
- net Gnd: now also Teensy1.G3 (GND), Teensy1.G4 (GND), J3.1 (Pin_1), MAG1.2 (GND), PA1.8 (GND)
- net TX0: now reaches Teensy1.0
- net TX0: now also PA1.9 (TX0)
- net RX0: now reaches Teensy1.1
- net RX0: now also PA1.10 (RX0)
- net SCL: now reaches Teensy1.24
- net SCL: now also MAG1.3 (SCL)
- net SDA: now reaches Teensy1.25
- net SDA: now also MAG1.4 (SDA)
- net 3.3V: now reaches Teensy1.V2 (3.3V)
- net 3.3V: now also MAG1.1 (Vcc), PA1.1 (Vcc)
- new net: J2.1 (Pin_1), PA1.11 (EX_ANT)
- new net: J1.1 (Pin_1), MAG1.5 (DRDY)
- now unconnected: Teensy1.~ (GND), Teensy1.~ (GND), Teensy1.~ (GND), Teensy1.~ (GND)
Other:
- moved on the sheet: R1, R10, R2, R3, R4, R5, R6, R7, R8, R9, TOF1, TOF2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

Commit message: Made sensors work
Parts:
- removed J1, J2, J3: Conn_01x01_Female, Custom_sym:1x1 Pad, symbol Connector:Conn_01x01_Female
- removed MAG1: Magnetometer, Custom_sym:Magnetometer, symbol custom_sym:Magnetometer
- added Ant1: SMAAntennaMale, Custom_sym:SMAAntennaMale, symbol custom_sym:SMAAntennaMale
- added DC-DC1: BuckConverter(LM2596), Custom_sym:BuckConverter(LM2596), symbol custom_sym:BuckConverter(LM2596)
- added Debug1: RaspberryPiDebug, symbol custom_sym:RaspberryPiDebug
- added Rasp1: RaspberryPi3, Custom_sym:RasberryPI3, symbol custom_sym:RaspberryPi3
- added U1: ExternalBattery, Custom_sym:ExternalBattery, symbol custom_sym:ExternalBattery
- added U2, U3: 1×24, Custom_sym:1×24, symbol custom_sym:1×24
- added XH-3A1, XH-3A2, XH-3A3, XH-3A4: XH-3AFemaleConnector, Custom_sym:XH-3A Female Connector, symbol custom_sym:XH-3AFemaleConnector
Connections:
- net 3.3V: now also U2.15
- net RX0: now also U2.3
- net SCL: now also U2.16
- net SDA: now also U2.17
- net TX0: now also U2.2
- net Trig1: now also U3.20
- net Trig2: now also U3.22
- net Trig3: now also U3.24
- net Trig4: now also U2.23
- net Trig5: now also U2.21
- net TOF2: now reaches R2.2, R4.1, Teensy1.30
- net TOF2: now also U2.22
- net TOF1: now reaches R1.2, R3.1, Teensy1.32
- net TOF1: now also U2.24
- net TOF5: now reaches R10.2, R9.1, Teensy1.34
- net TOF5: now also U3.23
- net TOF4: now reaches R6.1, R8.2, Teensy1.36
- net TOF4: now also U3.21
- net TOF3: now reaches R5.1, R7.2, Teensy1.38
- net TOF3: now also U3.19
- net at PA1.11 (EX_ANT): now also Ant1.1 (Antenna_IN)
- net Gnd renamed GND
- net GND: now also Ant1.Gnd, DC-DC1.OUT-, Debug1.14, Debug1.20, Debug1.25, Debug1.30, Debug1.34, Debug1.39, Debug1.6, Debug1.9, Rasp1.14 (GND), Rasp1.20 (GND), Rasp1.25 (GND), Rasp1.30 (GND), Rasp1.34 (GND), Rasp1.39 (GND), Rasp1.6 (GND), Rasp1.9 (GND), U2.1, U3.15, U3.2, XH-3A1.1, XH-3A2.1, XH-3A3.1, XH-3A4.1
- net Vin renamed 5V
- net 5V: now also DC-DC1.OUT+, Debug1.2, Debug1.4, Rasp1.2 (5V), Rasp1.4 (5V), U3.1
- new net: DC-DC1.IN+ (‌IN+), U1.VBattery (OUT+)
- new net: DC-DC1.IN-, U1.GND (OUT-)
- new net DIR1: Debug1.16, Rasp1.16 (GPIO_23), XH-3A1.3, XH-3A2.3
- new net DIR2: Debug1.18, Rasp1.18 (GPIO_24), XH-3A3.3, XH-3A4.3
- new net PWMLeft: Debug1.32, Rasp1.32 (GPIO_12), XH-3A1.2, XH-3A2.2
- new net PWMRight: Debug1.33, Rasp1.33 (GPIO_13), XH-3A3.2, XH-3A4.2
Other:
- moved on the sheet: PA1, R1, R10, R2, R3, R4, R5, R6, R7, R8, R9, TOF1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

Commit message: pcb design 3.0
Parts:
- added U4: ExternalBattery, Custom_sym:BatteryBackUp, symbol custom_sym:ExternalBattery
- Debug1: footprint (none) -> Custom_sym:2×20
- R1, R10, R2, R3, R4, R5, R6, R7, R8, R9: footprint Resistors_THT:R_Axial_DIN0207_L6.3mm_D2.5mm_P10.16mm_Horizontal -> Custom_sym:Resistor
Connections:
- net GND: now also U4.GND (OUT-)
- net TOF4: now also Teensy1.39, U3.18; no longer Teensy1.36, U3.21
- net Trig2: now also Teensy1.36, U3.21; no longer Teensy1.35, U3.22
- net Trig4: now also Teensy1.29, U2.21; no longer Teensy1.31, U2.23
- net Trig5: now also Teensy1.28, U2.20; no longer Teensy1.29, U2.21
- net at Teensy1.10: now also U2.12
- net at Teensy1.11: now also U2.13
- net at Teensy1.12: now also U2.14
- net at Teensy1.13: now also U3.14
- net at Teensy1.14: now also U3.13
- net at Teensy1.15: now also U3.12
- net at Teensy1.16: now also U3.11
- net at Teensy1.17: now also U3.10
- net at Teensy1.18: now also U3.9
- net at Teensy1.19: now also U3.8
- net at Teensy1.2: now also U2.4
- net at Teensy1.20: now also U3.7
- net at Teensy1.21: now also U3.6
- net at Teensy1.22: now also U3.5
- net at Teensy1.23: now also U3.4
- net at Teensy1.26: now also U2.18
- net at Teensy1.27: now also U2.19
- net at Teensy1.3: now also U2.5
- net at Teensy1.4: now also U2.6
- net at Teensy1.40: now also U3.17
- net at Teensy1.41: now also U3.16
- net at Teensy1.5: now also U2.7
- net at Teensy1.6: now also U2.8
- net at Teensy1.7: now also U2.9
- net at Teensy1.8: now also U2.10
- net at Teensy1.9: now also U2.11
- net at Teensy1.V1 (3.3V): now also U3.3
- net VBattery: now reaches PA1.4 (VBackUp)
- net VBattery: now also U4.VBattery (OUT+)
- net 1: now reaches Rasp1.1 (3.3V)
- net 1: now also Debug1.1
- net at Rasp1.10 (UARTO_RX): now also Debug1.10
- net 11: now reaches Rasp1.11 (GPIO_17)
- net 11: now also Debug1.11
- net at Rasp1.12 (GPIO_18): now also Debug1.12
- net 13: now reaches Rasp1.13 (GPIO_27)
- net 13: now also Debug1.13
- net 15: now reaches Rasp1.15 (GPIO_22)
- net 15: now also Debug1.15
- net 17: now reaches Rasp1.17 (3.3V)
- net 17: now also Debug1.17
- net 19: now reaches Rasp1.19 (GPIO_10)
- net 19: now also Debug1.19
- net 21: now reaches Rasp1.21 (GPIO_9)
- net 21: now also Debug1.21
- net at Rasp1.22 (GPIO_25): now also Debug1.22
- net 23: now reaches Rasp1.23 (GPIO_11)
- net 23: now also Debug1.23
- net at Rasp1.24 (GPIO_8): now also Debug1.24
- net at Rasp1.26 (GPIO_7): now also Debug1.26
- net 27: now reaches Rasp1.27 (Reserved)
- net 27: now also Debug1.27
- net at Rasp1.28 (Reserved): now also Debug1.28
- net 29: now reaches Rasp1.29 (GPIO_5)
- net 29: now also Debug1.29
- net 3: now reaches Rasp1.3 (GPIO_2)
- net 3: now also Debug1.3
- net 31: now reaches Rasp1.31 (GPIO_6)
- net 31: now also Debug1.31
- net 35: now reaches Rasp1.35 (GPIO_19)
- net 35: now also Debug1.35
- net at Rasp1.36 (GPIO_16): now also Debug1.36
- net 37: now reaches Rasp1.37 (GPIO_26)
- net 37: now also Debug1.37
- net at Rasp1.38 (GPIO_20): now also Debug1.38
- net at Rasp1.40 (GPIO_21): now also Debug1.40
- net 5: now reaches Rasp1.5 (GPIO_3)
- net 5: now also Debug1.5
- net 7: now reaches Rasp1.7 (GPIO_4)
- net 7: now also Debug1.7
- net at Rasp1.8 (UARTO_TX): now also Debug1.8
- new net: Teensy1.31, U2.23
- new net: Teensy1.35, U3.22
Other:
- moved on the sheet: Ant1, PA1
