File: kicad/gpsv1.1/gpsv1.3.kicad_pcb (KiCad board)
At the start: 2 copper layers, 200 x 120 mm, 35 parts, among them U1 ExternalBattery, U2 1×24, U3 1×24, U4 ExternalBattery

Commit message: Small changes to eliminate errors, and added buttons / leds
Parts:
- added B1: SW_Push, Custom_sym:button, F.Cu at (184.2, 139.7)
- added B2: SW_Push, Custom_sym:button, F.Cu at (175.8, 139.7)
- added B3: SW_Push, Custom_sym:button, F.Cu at (193.0, 139.7)
- added B4: SW_Push, Custom_sym:button, F.Cu at (167.6, 139.7)
- added LED1: LED, LED_THT:LED_D5.0mm_Clear, F.Cu at (94.0, 143.5)
- added LED2: LED, LED_THT:LED_D5.0mm_Clear, F.Cu at (101.6, 143.5)
- added LED3: LED, LED_THT:LED_D5.0mm_Clear, F.Cu at (109.2, 143.5)
- added LED4: LED, LED_THT:LED_D5.0mm_Clear, F.Cu at (116.8, 143.5)
- added R11: R, Custom_sym:Resistor, F.Cu at (96.5, 151.1)
- added R12: R, Custom_sym:Resistor, F.Cu at (104.1, 135.9)
- added R13: R, Custom_sym:Resistor, F.Cu at (111.1, 151.1)
- added R14: R, Custom_sym:Resistor, F.Cu at (127.0, 143.5)
- added R15: R, Custom_sym:Resistor, F.Cu at (181.6, 152.4)
- added R16: R, Custom_sym:Resistor, F.Cu at (173.4, 148.6)
- added R17: R, Custom_sym:Resistor, F.Cu at (190.5, 148.6)
- added R18: R, Custom_sym:Resistor, F.Cu at (158.8, 135.9)
Connections:
- net Net-(Debug1-Pad12) renamed 12
- net Net-(Debug1-Pad22) renamed 22
- net Net-(Debug1-Pad24) renamed 24
- net Net-(Debug1-Pad26) renamed 26
- net Net-(Debug1-Pad36) renamed 36
- net Net-(Debug1-Pad38) renamed 38
- net Net-(Debug1-Pad40) renamed 40
Routing:
- net 1: track 7.44 -> 126.7 mm, vias 0 -> 1
- net 40: track 7.07 -> 110.7 mm, vias 0 -> 7
- net 38: track 7.07 -> 95.8 mm, vias 0 -> 6
- net 36: track 7.07 -> 95.0 mm, vias 0 -> 3
- net 23: track 7.44 -> 88.2 mm, vias 0 -> 3
- net 22: track 7.07 -> 83.7 mm, vias 0 -> 1
- net 24: track 7.07 -> 83.3 mm, vias 0 -> 5
- net 26: track 7.07 -> 65.7 mm, vias 0 -> 1
- net 12: track 7.07 -> 42.3 mm, vias 0 -> 2
- net Trig4: track 106.9 -> 115.9 mm, vias 0 -> 2
- net 5V: track 16.8 -> 24.8 mm, vias 0 -> 1
- net Net-(LED3-Pad2): track 0.00 -> 7.88 mm
- net Net-(LED4-Pad2): track 0.00 -> 7.62 mm
- net Net-(LED2-Pad2): track 0.00 -> 7.62 mm
- net Net-(LED1-Pad2): track 0.00 -> 7.62 mm
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